Commit message: created a rough urdf model of the robot for further visualization and getting started with 3d cad design for raksh

File: ros2_ws/src/raksh_description/urdf/material.xacro (robot description, xacro)
@@ -1,6 +1,27 @@
 <?xml version="1.0"?>
-<robot xmlns:xacro="http://ros.org/wiki/xacro" name="raksh">
-    <material name="white">
-        <color rgba="1 1 1 1"></color>
-    </material>
+<robot>
+  <material name="black">
+    <color rgba="0.0 0.0 0.0 1.0"/>
+  </material>
+  <material name="white">
+    <color rgba="1.0 1.0 1.0 1.0"/>
+  </material>
+  <material name="red">
+    <color rgba="0.8 0.0 0.0 1.0"/>
+  </material>
+  <material name="blue">
+    <color rgba="0.0 0.0 0.8 1.0"/>
+  </material>
+  <material name="green">
+    <color rgba="0.0 0.8 0.0 1.0"/>
+  </material>
+  <material name="grey">
+    <color rgba="0.5 0.5 0.5 1.0"/>
+  </material>
+  <material name="orange">
+    <color rgba="${255/255} ${108/255} ${10/255} 1.0"/>
+  </material>
+  <material name="brown">
+    <color rgba="${222/255} ${207/255} ${195/255} 1.0"/>
+  </material>
 </robot>

File: ros2_ws/src/raksh_description/urdf/raksh.urdf.xacro (robot description, xacro)
@@ -1,4 +1,11 @@
 <?xml version="1.0"?>
 <robot xmlns:xacro="http://ros.org/wiki/xacro" name="raksh">
-    <xacro:include filename="raksh_core.xacro"/>
+    <xacro:include filename="$(find raksh_description)/urdf/material.xacro"/>
+    <xacro:include filename="$(find raksh_description)/urdf/raksh_description.urdf.xacro"/>
+    <link name="base_link"/>
+    <joint name="chasis_joint" type="fixed">
+        <origin xyz="-0.25 0 0" rpy="0 0 0"/>
+        <parent link="base_link"/>
+        <child link="chassis"/>
+    </joint>
 </robot>
